File: ESP8266_MainBoard/ESP8266_MainBoard.brd (EAGLE design)
At the start: 60 x 60 mm, 49 parts, among them IC1 PCF8574T, IC2 DS1820, IC3 4066D, IC4 DS2431P, Q1 BSS123, U2 PCF8575PWE4, X1 MICROMATCH-14, X2 MICROMATCH-6, X4 MICROMATCH-16, X5 MICROMATCH-4

Commit message: R13 von 4k7 nach 1k
Parts:
- R13: value 4k7 -> 1k
Changed lines of the file:
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@@
 <attribute name="NAME" x="41.148" y="14.351" size="1.27" layer="25"/>
 </element>
-<element name="R13" library="rcl" package="R0402" value="4k7" x="19.05" y="30.48" smashed="yes" rot="MR90">
+<element name="R13" library="rcl" package="R0402" value="1k" x="19.05" y="30.48" smashed="yes" rot="MR90">
 <attribute name="NAME" x="18.415" y="32.004" size="1.27" layer="26" rot="MR90"/>
 </element>
