File: ESP8266_MainBoard/ESP8266_MainBoard.sch (EAGLE design)
At the start: 49 parts, among them IC1 PCF8574T, IC2 DS1820, IC3 4066D, IC4 DS2431P, Q1 BSS123, U2 PCF8575PWE4, X1 MICROMATCH-14, X2 MICROMATCH-6, X4 MICROMATCH-16, X5 MICROMATCH-4

Commit message: R13 von 4k7 nach 1k
Parts:
- R13: value 4k7 -> 1k
Changed lines of the file:
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@@
 <part name="R11" library="rcl" deviceset="R-EU_" device="R0402" value="10k"/>
 <part name="R12" library="rcl" deviceset="R-EU_" device="R0402" value="10k"/>
-<part name="R13" library="rcl" deviceset="R-EU_" device="R0402" value="4k7"/>
+<part name="R13" library="rcl" deviceset="R-EU_" device="R0402" value="1k"/>
 <part name="+3V6" library="supply1" deviceset="+3V3" device=""/>
 <part name="+3V7" library="supply1" deviceset="+3V3" device=""/>
